File: Est. Met. V1.0.kicad_pcb (KiCad board)
At the start: 2 copper layers, 100 x 100 mm, 17 parts, among them J1 UART, J2 Pluv., J3 PWR, J4 S_Temp, Q1 2N7000, U1 StepDownLM2596, U2 ModuloA6_GSM, U3 BluePill_STM32F103

Commit message: Routeo con el modulo SIM800L
Parts:
- added D1: 1N4007, Diode_THT:D_DO-41_SOD81_P10.16mm_Horizontal, F.Cu at (114.7, 89.8)
- U2: value ModuloA6_GSM -> SIM800L_B; footprint My_Library:ModuloA6_GSM -> MyLibrary2:SIM800_B
- moved U2 17.9 mm to (124.6, 129.4), turned to 180 degrees
Connections:
- net MC_RST_A6 renamed MC_RST_S800
- J1 pad 2: RX_A6 -> RX_S800
- J1 pad 4: TX_A6 -> TX_S800
- Q1 pad 3: RST_A6 -> RST_S800
- U2 pad 1: +5V -> +4V
- U2 pad 2: GND -> RST_S800
- U2 pad 3: Net-(U2-Pad3) -> RX_S800
- U2 pad 4: Net-(U2-Pad4) -> TX_S800
- U2 pad 5: Net-(U2-Pad5) -> GND
- U2 pad 8: TX_A6 -> Net-(U2-Pad8)
- U2 pad 9: RX_A6 -> Net-(U2-Pad9)
- U3 pad 25: PWR_A6 -> Net-(U3-Pad25)
Routing:
- net PWR_A6: track 65.4 -> 0.00 mm
- net RST_A6: track 56.6 -> 0.00 mm
- net +4V: track 0.00 -> 53.8 mm
- net RST_S800: track 0.00 -> 43.3 mm
- net TX_S800: track 0.00 -> 42.6 mm
- net RX_S800: track 0.00 -> 40.6 mm
- net GND: track 73.5 -> 49.3 mm
- net +5V: track 98.5 -> 84.1 mm
- net TX_A6: track 13.4 -> 0.00 mm
- net RX_A6: track 13.4 -> 0.00 mm
Other:
- net class Default: trace_width 1 -> 1.27
- net class Señales: trace_width 0.8 -> 1; via_dia 0.5 -> 0.8

Commit message: Nueva placa
Parts:
- J1: value UART -> Conn_01x01; footprint Connector_PinHeader_2.54mm:PinHeader_1x06_P2.54mm_Vertical -> Connector_PinHeader_2.54mm:PinHeader_1x01_P2.54mm_Vertical
- moved U2 17.3 mm to (111.0, 118.7)
- moved J1 15.2 mm to (92.3, 107.6)
- moved C3 11.5 mm to (103.6, 81.9)
- moved C4 11.5 mm to (109.6, 81.9)
- moved D1 11.3 mm to (126.0, 89.4)
- moved C5 10.2 mm to (64.2, 67.2)
- moved C6 10.2 mm to (64.2, 61.2)
- moved J3 10.2 mm to (51.2, 69.2)
- moved U1 10.2 mm to (95.7, 65.2)
- moved Q1 3.61 mm to (96.4, 130.4)
Connections:
- J1 pad 1: TX_MC -> SWO
- U2 pad 4: TX_S800 -> RX_MC
- U3 pad 30: TX_MC -> RX_S800
Routing:
- net TX_S800: track 42.6 -> 0.00 mm
- net +4V: track 53.8 -> 25.9 mm
- net RX_MC: track 12.8 -> 40.7 mm
- net TX_MC: track 12.3 -> 0.00 mm
- net +5V: track 84.1 -> 74.3 mm
- net SWO: track 14.4 -> 6.47 mm
- net RST_S800: track 43.3 -> 37.4 mm
- net MC_RST_S800: track 14.3 -> 9.65 mm
Other:
- board size 100 x 100 mm -> 81.2 x 87.2 mm
