File: Est. Met. V1.0.sch (KiCad schematic (older format))
At the start: 17 parts, among them J1 UART, J2 Pluv., J3 PWR, J4 S_Temp, Q1 2N7000, U1 StepDownLM2596, U2 ModuloA6_GSM, U3 BluePill_STM32F103

Commit message: Routeo con el modulo SIM800L
Parts:
- removed U2: ModuloA6_GSM, My_Library:ModuloA6_GSM, symbol My_Library:ModuloA6_GSM
- added D1: 1N4007, Diode_THT:D_DO-41_SOD81_P10.16mm_Horizontal, symbol Diode:1N4007
- added U2: SIM800L_B, MyLibrary2:SIM800_B, symbol MyLibrary2:SIM800L_B
Connections:
- net +5V: now also D1.2 (A)
- net GND: now also U2.5 (GND)
- net MC_RST_A6 renamed MC_RST_S800
- net PWR_A6: no longer names the net of U3.25 (B12)
- net RST_A6 renamed RST_S800
- net RST_S800: now also U2.2 (RST)
- net RX_A6 renamed RX_S800
- net RX_S800: now also U2.3 (RXD)
- net TX_A6 renamed TX_S800
- net TX_S800: now also U2.4 (TXD)
- new net +4V: D1.1 (K), U2.1 (VCC_4.4V)
- no-connect marks 41 -> 36
Other:
- moved on the sheet: C1, C2, J1, J2, J4

Commit message: Nueva placa
Parts:
- removed J1: UART, Connector_PinHeader_2.54mm:PinHeader_1x06_P2.54mm_Vertical, symbol Connector_Generic:Conn_01x06
- added J1: Conn_01x01, Connector_PinHeader_2.54mm:PinHeader_1x01_P2.54mm_Vertical, symbol Connector_Generic:Conn_01x01
Connections:
- net TX_MC is gone; now on net RX_S800: U3.30 (A9)
- net TX_S800 is gone; now on net RX_MC: U2.4 (TXD)
- net SWO: now also J1.1 (Pin_1)
Changed lines of the file:
@@
 	3700 1900 3700 1625
-$Comp
-L power:GND #PWR0101
-U 1 1 5FDB5C8B
-P 8775 2675
-F 0 "#PWR0101" H 8775 2425 50  0001 C CNN
-F 1 "GND" H 8780 2502 50  0000 C CNN
-F 2 "" H 8775 2675 50  0001 C CNN
-F 3 "" H 8775 2675 50  0001 C CNN
-	1    8775 2675
-	1    0    0    -1
-$EndComp
 $Comp
 L power:PWR_FLAG #FLG0101
@@
 NoConn ~ 5925 5150
 NoConn ~ 5925 5050
-Wire Wire Line
-	8650 2250 8900 2250
-Wire Wire Line
-	8900 2150 8650 2150
-Wire Wire Line
-	8900 2050 8650 2050
-Wire Wire Line
-	8900 2350 8650 2350
-$Comp
-L Connector_Generic:Conn_01x06 J1
-U 1 1 5FE4F291
-P 8450 2150
-F 0 "J1" H 8450 1650 50  0000 C CNN
-F 1 "UART" H 8425 1725 50  0000 C CNN
-F 2 "Connector_PinHeader_2.54mm:PinHeader_1x06_P2.54mm_Vertical" H 8450 2150 50  0001 C CNN
-F 3 "~" H 8450 2150 50  0001 C CNN
-	1    8450 2150
-	-1   0    0    1
-$EndComp
-Wire Wire Line
-	8775 1850 8650 1850
-Wire Wire Line
-	8775 1850 8775 2675
 Text GLabel 4275 5250 0    50   Input ~ 0
 SWO
 Wire Wire Line
 	4275 5250 4625 5250
-Text GLabel 8900 1950 2    50   Input ~ 0
+Text GLabel 9200 1600 2    50   Input ~ 0
 SWO
-Wire Wire Line
-	8900 1950 8650 1950
 Wire Wire Line
 	2600 5200 2600 5050
@@
 	4075 1625 4075 1900
 Connection ~ 4075 1900
+$Comp
+L Connector_Generic:Conn_01x01 J1
+U 1 1 620EF853
+P 8875 1600
+F 0 "J1" H 8793 1375 50  0000 C CNN
+F 1 "Conn_01x01" H 8793 1466 50  0000 C CNN
+F 2 "Connector_PinHeader_2.54mm:PinHeader_1x01_P2.54mm_Vertical" H 8875 1600 50  0001 C CNN
+F 3 "~" H 8875 1600 50  0001 C CNN
+	1    8875 1600
+	-1   0    0    1
+$EndComp
+Wire Wire Line
+	8825 2250 8900 2250
+Wire Wire Line
+	8825 2350 8825 2250
+Wire Wire Line
+	8900 2350 8825 2350
+Wire Wire Line
+	8825 2050 8900 2050
+Wire Wire Line
+	8825 2150 8825 2050
+Wire Wire Line
+	8900 2150 8825 2150
+Wire Wire Line
+	9075 1600 9200 1600
 $EndSCHEMATC
